File: hardware/fancontrol.brd (EAGLE design)
At the start: 55 x 50 mm, 13 parts, among them Q1 IRLZ44Z, T1 BC547

Commit message: New pcb layout
+ new pdf files.
Parts:
- removed C1: 470u, rcl:E5-10,5
- removed Q1: IRLZ44Z, transistor-power:TO220BH
- removed R2: 10R, rcl:0207/7
- removed R3: 10k, rcl:0207/7
- removed T1: BC547, transistor:TO92
- added D1: 1N4004, diode:DO41-10
- added T2: BD535, transistor:TO220
- R1: value 10k -> 220
- moved C3 17.6 mm to (9.35, 6.26)
- moved R4 9.96 mm to (36.5, 26.0), turned to 0 degrees
- moved C2 7.79 mm to (14.4, 6.26)
- moved JP2 7.73 mm to (22.6, 6.27)
- moved R1 2.01 mm to (40.8, 17.4)
- moved JP1 0.07 mm to (40.0, 6.07), turned to 180 degrees
Connections:
- removed net FAN+: C1.+, JP2.1, Q1.S
- removed net N$3: Q1.G, R2.2, R3.2
- net +12V: now also D1.C, JP2.1; no longer Q1.D, R3.1
- net GND: now also T2.1; no longer C1.-, JP2.3, T1.1
- net N$1: now also D1.A, JP2.3, T2.2; no longer R1.2, T1.2
- net N$2: now also R1.2, T2.3; no longer R2.1, T1.3
Routing:
- net FAN+: track 44.3 -> 0.00 mm
- net +5V: track 92.5 -> 60.3 mm
- net +12V: track 58.9 -> 38.1 mm
- net N$3: track 17.0 -> 0.00 mm
- net N$1: track 9.06 -> 22.8 mm
- net N$2: track 7.69 -> 17.5 mm
- net DQ: track 25.6 -> 31.5 mm
- net PWM: track 5.51 -> 7.42 mm
- net TACHO: track 66.3 -> 65.5 mm
Other:
- board size 55 x 50 mm -> 55 x 49.8 mm
