File: hardware/fancontrol.sch (EAGLE design)
At the start: 10 parts, among them T2 BD535

Commit message: New pcb layout
+ new pdf files.
Parts:
- R1: value (none) -> 220
Changed lines of the file:
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@@
 <part name="P+2" library="supply1" deviceset="+12V" device=""/>
 <part name="GND1" library="supply1" deviceset="GND" device=""/>
-<part name="R1" library="rcl" deviceset="R-EU_" device="0207/7"/>
+<part name="R1" library="rcl" deviceset="R-EU_" device="0207/7" value="220"/>
 <part name="ARDUINO1" library="arduino" deviceset="ARDUINO" device=""/>
 <part name="GND3" library="supply1" deviceset="GND" device=""/>
